Commit message: with simplified collisions

File: msj_platform/model.urdf (robot description, URDF)
Before this commit: robot msj_platform, 4 links, 3 joints
Links:
- link base: geometry collision mesh filename=package://robots/msj_platform/meshes/collisions/base.dae scale=0.001 0.001 0.001; visual mesh filename=package://robots/msj_platform/meshes/visuals/base.dae scale=0.001 0.001 0.001
- link sphere_link1: geometry collision mesh filename=package://robots/msj_platform/meshes/collisions/sphere_link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 scale=0.001 0.001 0.001; visual mesh filename=package://robots/msj_platform/meshes/visuals/sphere_link1.d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 scale=0.001 0.001 0.001
- link sphere_link2: geometry collision mesh filename=package://robots/msj_platform/meshes/collisions/sphere_link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 scale=0.001 0.001 0.001; visual mesh filename=package://robots/msj_platform/meshes/visuals/sphere_link2.d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 scale=0.001 0.001 0.001
- link top: geometry collision mesh filename=package://robots/msj_platform/meshes/collisions/top.dae scale=0.001 0.001 0.001; visual mesh filename=package://robots/msj_platform/meshes/visuals/top.dae scale=0.001 0.001 0.001
Joints:
- joint sphere_axis0: axis 1 0 0 -> 1  0  0; origin xyz=0.00757 -0.006    0.108 rpy=0 0 0 -> xyz=0.00757 -0.006    0.108 rpy=0  0  0
- joint sphere_axis1: axis 0 1 0 -> 0  1  0; origin xyz=0 0 0 rpy=0 0 0 -> xyz=0  0  0 rpy=0  0  0
- joint sphere_axis2: axis 0 0 1 -> 0  0  1; origin xyz=0 0 0 rpy=0 0 0 -> xyz=0  0  0 rpy=0  0  0
